File: EnvMon.kicad_pcb (KiCad board)
At the start: 2 copper layers, 28 x 39 mm, 10 parts, among them J1 Power, J2 TFT, J3 AE-BME280, J4 MH-Z19B, J5 STM32_Debug, U1 STM32F303K8Tx

Commit message: 基板 V2.0
Parts:
- removed SW: SW_Push, EnvMon:SW-2pin
- added C3: 0.1uF, Capacitor_SMD:C_0603_1608Metric_Pad1.05x0.95mm_HandSolder, F.Cu at (-4.30, 15.7)
- added D1: BT_Connect, LED_SMD:LED_0603_1608Metric_Pad1.05x0.95mm_HandSolder, F.Cu at (-11.8, 13.8)
- added R2: 10k, Resistor_SMD:R_0603_1608Metric_Pad1.05x0.95mm_HandSolder, F.Cu at (-8.03, 15.7)
- added R3: 10k, Resistor_SMD:R_0603_1608Metric_Pad1.05x0.95mm_HandSolder, F.Cu at (-8.03, 13.8)
- added R4: 1k, Resistor_SMD:R_0603_1608Metric_Pad1.05x0.95mm_HandSolder, F.Cu at (-11.8, 15.7)
- added SW1: TouchSW, EnvMon:TouchSW, F.Cu at (6.63, 4.00)
- added U2: RN4020, EnvMon:RN4020, F.Cu at (6.10, 30.0)
- moved C2 8.95 mm to (6.78, 15.4)
- moved U1 8.46 mm to (1.52, 11.2)
- moved C1 6.31 mm to (-5.96, 8.40)
- moved R1 6.09 mm to (-5.96, 6.50), turned to 180 degrees
- moved J4 0.11 mm to (-10.3, 18.6)
Connections:
- U1 pad 10: (no net) -> RN4020_WAKE
- U1 pad 21: (no net) -> TFT_RES
- U1 pad 22: (no net) -> TFT_DC
- U1 pad 28: (no net) -> TFT_BLK
- U1 pad 7: TFT_BLK -> (no net)
- U1 pad 8: TFT_DC -> USART2_TX
- U1 pad 9: TFT_RES -> USART2_RX
Routing:
- net GND: track 36.0 -> 130.2 mm
- net USART1_TX: track 45.0 -> 17.2 mm
- net TFT_RES: track 36.7 -> 11.1 mm, vias 2 -> 1
- net USART1_RX: track 39.6 -> 14.5 mm
- net TFT_DC: track 32.7 -> 10.00 mm, vias 2 -> 1
- net Net-(R4-Pad2): track 0.00 -> 22.2 mm, vias 0 -> 2
- net Net-(R3-Pad2): track 0.00 -> 21.5 mm
- net DISP_SW: track 36.4 -> 15.3 mm
- net TFT_BLK: track 32.4 -> 12.4 mm, vias 2 -> 0
- net Net-(R2-Pad1): track 0.00 -> 19.0 mm
- net USART2_TX: track 0.00 -> 18.7 mm, vias 0 -> 2
- net USART2_RX: track 0.00 -> 18.5 mm, vias 0 -> 2
- net +3V3: track 76.5 -> 90.2 mm
- net RN4020_WAKE: track 0.00 -> 10.8 mm
- net SPI1_MOSI: track 24.8 -> 15.0 mm, vias 2 -> 1
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Other:
- net class Default: via_dia 0.508 -> 0.6096; via_drill 0.254 -> 0.3048
- net class Power added: clearance 0.2032, trace_width 0.254, via_dia 0.6096, via_drill 0.3048
- rule via_min_drill: 0.254 -> 0.3048
- rule via_min_size: 0.508 -> 0.6096
- board text added: "EnvMonBT V2.0"
- board text removed: "EnvMon V1.0"

Commit message: 基板 V2.1
Parts:
- added C4: 10pF, EnvMon:C_0402_1005Metric, F.Cu at (-9.19, 7.90)
- added C5: 10pF, EnvMon:C_0402_1005Metric, F.Cu at (-5.49, 12.2)
- added X1: 12MHz, EnvMon:Crystal_SMD_3225-4Pin_3.2x2.5mm_HandSoldering, F.Cu at (-5.80, 9.20)
- moved C1 2.74 mm to (-7.28, 6.00)
- moved R1 2.22 mm to (-3.77, 6.10)
Connections:
- U1 pad 2: (no net) -> OSC_IN
- U1 pad 3: (no net) -> OSC_OUT
Routing:
- net +3V3: track 90.2 -> 106.6 mm, vias 0 -> 1
- net GND: track 130.2 -> 139.3 mm
- net OSC_IN: track 0.00 -> 7.09 mm
- net OSC_OUT: track 0.00 -> 4.04 mm
- net Net-(R1-Pad1): track 6.08 -> 4.45 mm
Other:
- board text added: "EnvMonBT V2.1"
- board text removed: "EnvMonBT V2.0"
