File: EnvMon.sch (KiCad schematic (older format))
At the start: 10 parts, among them J1 Power, J2 TFT, J3 AE-BME280, J4 MH-Z19B, J5 STM32_Debug, SW1 SW_Push, U1 STM32F303K8Tx

Commit message: 基板 V2.0
Parts:
- removed SW1: SW_Push, EnvMon:SW-2pin, symbol Switch:SW_Push
- added C3: 0.1uF, Capacitor_SMD:C_0603_1608Metric_Pad1.05x0.95mm_HandSolder, symbol Device:C_Small
- added D1: BT_Connect, LED_SMD:LED_0603_1608Metric_Pad1.05x0.95mm_HandSolder, symbol Device:LED_Small
- added R2, R3: 10k, Resistor_SMD:R_0603_1608Metric_Pad1.05x0.95mm_HandSolder, symbol Device:R
- added R4: 1k, Resistor_SMD:R_0603_1608Metric_Pad1.05x0.95mm_HandSolder, symbol Device:R
- added SW1: TouchSW, EnvMon:TouchSW, symbol EnvMon:TouchSW
- added U2: RN4020, EnvMon:RN4020, symbol EnvMon:RN4020
Connections:
- net labels added: RN4020_WAKE, USART2_RX, USART2_TX
- wire segments 40 -> 60
- no-connect marks 15 -> 22
Other:
- moved on the sheet: C1, C2, J1, J2, J3, J4, J5, R1, U1

Commit message: 基板 V2.1
Parts:
- added C4, C5: 10pF, EnvMon:C_0402_1005Metric, symbol Device:C_Small
- added X1: 12MHz, EnvMon:Crystal_SMD_3225-4Pin_3.2x2.5mm_HandSoldering, symbol Device:Crystal_GND24_Small
Connections:
- net GND: now also C4.2, C5.2, X1.2, X1.4
- net OSC_IN: now reaches U1.2 (PF0)
- net OSC_IN: now also C4.1, X1.1
- net OSC_OUT: now reaches U1.3 (PF1)
- net OSC_OUT: now also C5.1, X1.3
- no-connect marks 22 -> 20
Changed lines of the file:
@@
 Sheet 1 1
 Title "EnvMonBT"
-Date "2020-10-11"
-Rev "2.0"
+Date "2021-01-14"
+Rev "2.1"
 Comp ""
 Comment1 ""
@@
 	4900 2250 4600 2250
 Wire Wire Line
-	4900 2650 4600 2650
-Wire Wire Line
-	4600 2650 4600 2250
-Connection ~ 4600 2250
+	4500 2650 4500 2250
 $Comp
 L power:GND #PWR011
@@
 NoConn ~ 5850 3300
 NoConn ~ 6300 2850
-NoConn ~ 4900 2450
-NoConn ~ 4900 2350
 Text GLabel 8100 2750 0    50   Input ~ 0
 SWDIO
@@
 	-1   0    0    1
 $EndComp
+$Comp
+L Device:Crystal_GND24_Small X1
+U 1 1 6000954A
+P 3750 1100
+F 0 "X1" H 3800 1300 50  0000 L CNN
+F 1 "12MHz" H 3800 1200 50  0000 L CNN
+F 2 "EnvMon:Crystal_SMD_3225-4Pin_3.2x2.5mm_HandSoldering" H 3750 1100 50  0001 C CNN
+F 3 "~" H 3750 1100 50  0001 C CNN
+	1    3750 1100
+	1    0    0    -1
+$EndComp
+Text GLabel 4900 2350 0    50   Input ~ 0
+OSC_IN
+Text GLabel 4900 2450 0    50   Input ~ 0
+OSC_OUT
+Wire Wire Line
+	4600 2250 4500 2250
+Connection ~ 4600 2250
+Wire Wire Line
+	4500 2650 4900 2650
+Text GLabel 3450 1100 0    50   Input ~ 0
+OSC_IN
+Text GLabel 4050 1100 2    50   Input ~ 0
+OSC_OUT
+$Comp
+L power:GND #PWR018
+U 1 1 60012320
+P 3750 1350
+F 0 "#PWR018" H 3750 1100 50  0001 C CNN
+F 1 "GND" H 3750 1200 50  0000 C CNN
+F 2 "" H 3750 1350 50  0001 C CNN
+F 3 "" H 3750 1350 50  0001 C CNN
+	1    3750 1350
+	1    0    0    -1
+$EndComp
+$Comp
+L Device:C_Small C4
+U 1 1 60015B42
+P 3550 1250
+F 0 "C4" H 3350 1300 50  0000 L CNN
+F 1 "10pF" H 3250 1200 50  0000 L CNN
+F 2 "EnvMon:C_0402_1005Metric" H 3550 1250 50  0001 C CNN
+F 3 "~" H 3550 1250 50  0001 C CNN
+	1    3550 1250
+	1    0    0    -1
+$EndComp
+$Comp
+L Device:C_Small C5
+U 1 1 60017276
+P 3950 1250
+F 0 "C5" H 4050 1300 50  0000 L CNN
+F 1 "10pF" H 4050 1200 50  0000 L CNN
+F 2 "EnvMon:C_0402_1005Metric" H 3950 1250 50  0001 C CNN
+F 3 "~" H 3950 1250 50  0001 C CNN
+	1    3950 1250
+	1    0    0    -1
+$EndComp
+Wire Wire Line
+	3550 1100 3650 1100
+Connection ~ 3550 1100
+Wire Wire Line
+	3550 1100 3550 1150
+Wire Wire Line
+	3550 1100 3450 1100
+Wire Wire Line
+	3850 1100 3950 1100
+Wire Wire Line
+	3950 1100 3950 1150
+Connection ~ 3950 1100
+Wire Wire Line
+	3950 1100 4050 1100
+Wire Wire Line
+	3950 1350 3750 1350
+Wire Wire Line
+	3750 1350 3550 1350
+Connection ~ 3750 1350
+$Comp
+L power:GND #PWR017
+U 1 1 6002D116
+P 3550 850
+F 0 "#PWR017" H 3550 600 50  0001 C CNN
+F 1 "GND" H 3550 700 50  0000 C CNN
+F 2 "" H 3550 850 50  0001 C CNN
+F 3 "" H 3550 850 50  0001 C CNN
+	1    3550 850
+	1    0    0    -1
+$EndComp
+Wire Wire Line
+	3550 850  3750 850
+Wire Wire Line
+	3750 850  3750 1000
+Wire Wire Line
+	3750 1200 3750 1350
 $EndSCHEMATC
